Commit message: Updates for new power system

File: mushr_description/robots/mushr_tx2.urdf.xacro (robot description, xacro)
@@ -11,5 +11,5 @@
 	<xacro:mushr_ydlidar />
 	<xacro:sensor_d435 parent="base_link" >
-  		<origin xyz="0.10075 0.0 0.0945" rpy="0 0 0" />
+  		<origin xyz="0.10075 0.0 0.099" rpy="0 0 0" />
 	</xacro:sensor_d435>
 	<link name="front_left/wheel_steer_link"/>
@@ -107,5 +107,5 @@
 		type="fixed" >
 		<origin
-			xyz="-0.038975 0 0.15325"
+			xyz="-0.038975 0 0.15775"
 			rpy="0 0 0" />
 		<parent
