Commit message: Added files to allow URDF generation of different colored cars

File: mushr_description/robots/mushr_base_nano.urdf.xacro (robot description, xacro)
@@ -37,5 +37,5 @@
 					rpy="0 0 0" />
 				<geometry>
-					<mesh filename="package://mushr_description/meshes/base/mushr_base_nano.dae" />
+					<mesh filename="package://mushr_description/meshes/base/nano/mushr_base_nano.dae" />
 				</geometry>
 			</visual>
@@ -45,5 +45,5 @@
 					rpy="0 0 0" />
 				<geometry>
-					<mesh filename="package://mushr_description/meshes/base/mushr_base_collision_nano.dae" />
+					<mesh filename="package://mushr_description/meshes/base/nano/mushr_base_nano_collision.dae" />
 				</geometry>
 			</collision>

File: mushr_description/robots/mushr_base_tx2.urdf.xacro (robot description, xacro)
@@ -37,5 +37,5 @@
 					rpy="0 0 0" />
 				<geometry>
-					<mesh filename="package://mushr_description/meshes/base/mushr_base_tx2.dae" />
+					<mesh filename="package://mushr_description/meshes/base/tx2/mushr_base_tx2.dae" />
 				</geometry>
 			</visual>
@@ -45,5 +45,5 @@
 					rpy="0 0 0" />
 				<geometry>
-					<mesh filename="package://mushr_description/meshes/base/mushr_base_collision_tx2.dae" />
+					<mesh filename="package://mushr_description/meshes/base/tx2/mushr_base_tx2_collision.dae" />
 				</geometry>
 			</collision>

Commit message: CMakeLists.txt

File: mushr_description/robots/mushr_base_nano.urdf.xacro (robot description, xacro)
@@ -1,4 +1,5 @@
 <robot xmlns:xacro="http://ros.org/wiki/xacro" name="mushr_base_nano">
-	<xacro:macro name="mushr_base_nano">
+	<xacro:include filename="color.urdf.xacro" />
+	<xacro:macro name="mushr_base_nano" params="platform_color:=none inset_color:=none">
 		<link name="base_footprint">
 			<inertial>
@@ -32,20 +33,110 @@
 					izz="1" />
 			</inertial>
+			<xacro:if value="${platform_color == 'none' and inset_color == 'none'}">
 			<visual>
+					<origin
+						xyz="0 0 0"
+						rpy="0 0 0" />
+					<geometry>
+						<mesh filename="package://mushr_description/meshes/base/nano/mushr_base_nano.dae" />
+					</geometry>
+				</visual>
+				<collision>
+					<origin
+						xyz="0 0 0"
+						rpy="0 0 0" />
+					<geometry>
+						<mesh filename="package://mushr_description/meshes/base/nano/mushr_base_nano_collision.dae" />
+					</geometry>
+				</collision>
+			</xacro:if>
+			<xacro:unless value="${platform_color == 'none' and inset_color == 'none'}">
+				<visual>
+					<origin
+						xyz="0 0 0"
+						rpy="0 0 0" />
+					<geometry>
+						<mesh filename="package://mushr_description/meshes/base/nano/mushr_base_nano_core.dae" />
+					</geometry>
+				</visual>
+				<collision>
+					<origin
+						xyz="0 0 0"
+						rpy="0 0 0" />
+					<geometry>
+						<mesh filename="package://mushr_description/meshes/base/nano/mushr_base_nano_core_collision.dae" />
+					</geometry>
+				</collision>
+			</xacro:unless>
+		</link>
+		<link name="platform_link">
+			<inertial>
 				<origin
 					xyz="0 0 0"
 					rpy="0 0 0" />
-				<geometry>
-					<mesh filename="package://mushr_description/meshes/base/nano/mushr_base_nano.dae" />
-				</geometry>
-			</visual>
-			<collision>
+				<mass
+					value="1.0" />
+				<inertia
+					ixx="1"
+					ixy="0"
+					ixz="0"
+					iyy="1"
+					iyz="0"
+					izz="1" />
+			</inertial>
+			<xacro:unless value="${platform_color == 'none' and inset_color == 'none'}">
+				<visual>
+					<origin
+						xyz="0 0 0"
+						rpy="0 0 0" />
+					<geometry>
+						<mesh filename="package://mushr_description/meshes/base/nano/mushr_base_nano_platform.stl" />
+					</geometry>
+					<material name="${platform_color}"/>
+				</visual>
+				<collision>
+					<origin
+						xyz="0 0 0"
+						rpy="0 0 0" />
+					<geometry>
+						<mesh filename="package://mushr_description/meshes/base/nano/mushr_base_nano_platform_collision.dae" />
+					</geometry>
+				</collision>
+			</xacro:unless>
+		</link>
+		<link name="insets_link">
+			<inertial>
 				<origin
 					xyz="0 0 0"
 					rpy="0 0 0" />
-				<geometry>
-					<mesh filename="package://mushr_description/meshes/base/nano/mushr_base_nano_collision.dae" />
-				</geometry>
-			</collision>
+				<mass
+					value="1.0" />
+				<inertia
+					ixx="1"
+					ixy="0"
+					ixz="0"
+					iyy="1"
+					iyz="0"
+					izz="1" />
+			</inertial>
+			<xacro:unless value="${platform_color == 'none' and inset_color == 'none'}">
+				<visual>
+					<origin
+						xyz="0 0 0"
+						rpy="0 0 0" />
+					<geometry>
+						<mesh filename="package://mushr_description/meshes/base/nano/mushr_base_nano_insets.stl" />
+					</geometry>
+					<material name="${inset_color}"/>
+				</visual>
+				<collision>
+					<origin
+						xyz="0 0 0"
+						rpy="0 0 0" />
+					<geometry>
+						<mesh filename="package://mushr_description/meshes/base/nano/mushr_base_nano_insets_collision.dae" />
+					</geometry>
+				</collision>
+			</xacro:unless>
 		</link>
 		<joint
@@ -60,4 +151,26 @@
 				link="base_link" />
 		</joint>
+		<joint
+			name="base_link_to_platform_link"
+			type="fixed">
+			<origin
+				xyz="0 0 0.0"
+				rpy="0 0 0" />
+			<parent
+				link="base_link" />
+			<child
+				link="platform_link" />
+		</joint>
+		<joint
+			name="base_link_to_insets_link"
+			type="fixed">
+			<origin
+				xyz="0 0 0.0"
+				rpy="0 0 0" />
+			<parent
+				link="base_link" />
+			<child
+				link="insets_link" />
+		</joint>
 	</xacro:macro>
 </robot>

File: mushr_description/robots/mushr_base_tx2.urdf.xacro (robot description, xacro)
@@ -1,4 +1,5 @@
 <robot xmlns:xacro="http://ros.org/wiki/xacro" name="mushr_base_tx2">
-	<xacro:macro name="mushr_base_tx2">
+	<xacro:include filename="color.urdf.xacro" />
+	<xacro:macro name="mushr_base_tx2" params="platform_color:=none inset_color:=none">
 		<link name="base_footprint">
 			<inertial>
@@ -32,20 +33,110 @@
 					izz="1" />
 			</inertial>
-			<visual>
+			<xacro:if value="${platform_color == 'none' and inset_color == 'none'}">
+				<visual>
+					<origin
+						xyz="0 0 0"
+						rpy="0 0 0" />
+					<geometry>
+						<mesh filename="package://mushr_description/meshes/base/tx2/mushr_base_tx2.dae" />
+					</geometry>
+				</visual>
+				<collision>
+					<origin
+						xyz="0 0 0"
+						rpy="0 0 0" />
+					<geometry>
+						<mesh filename="package://mushr_description/meshes/base/tx2/mushr_base_tx2_collision.dae" />
+					</geometry>
+				</collision>
+			</xacro:if>
+			<xacro:unless value="${platform_color == 'none' and inset_color == 'none'}">
+				<visual>
+					<origin
+						xyz="0 0 0"
+						rpy="0 0 0" />
+					<geometry>
+						<mesh filename="package://mushr_description/meshes/base/tx2/mushr_base_tx2_core.dae" />
+					</geometry>
+				</visual>
+				<collision>
+					<origin
+						xyz="0 0 0"
+						rpy="0 0 0" />
+					<geometry>
+						<mesh filename="package://mushr_description/meshes/base/tx2/mushr_base_tx2_core_collision.dae" />
+					</geometry>
+				</collision>
+			</xacro:unless>
+		</link>
+		<link name="platform_link">
+			<inertial>
 				<origin
 					xyz="0 0 0"
 					rpy="0 0 0" />
-				<geometry>
-					<mesh filename="package://mushr_description/meshes/base/tx2/mushr_base_tx2.dae" />
-				</geometry>
-			</visual>
-			<collision>
+				<mass
+					value="1.0" />
+				<inertia
+					ixx="1"
+					ixy="0"
+					ixz="0"
+					iyy="1"
+					iyz="0"
+					izz="1" />
+			</inertial>
+			<xacro:unless value="${platform_color == 'none' and inset_color == 'none'}">
+				<visual>
+					<origin
+						xyz="0 0 0"
+						rpy="0 0 0" />
+					<geometry>
+						<mesh filename="package://mushr_description/meshes/base/tx2/mushr_base_tx2_platform.stl" />
+					</geometry>
+					<material name="${platform_color}"/>
+				</visual>
+				<collision>
+					<origin
+						xyz="0 0 0"
+						rpy="0 0 0" />
+					<geometry>
+						<mesh filename="package://mushr_description/meshes/base/tx2/mushr_base_tx2_platform_collision.dae" />
+					</geometry>
+				</collision>
+			</xacro:unless>
+		</link>
+		<link name="insets_link">
+			<inertial>
 				<origin
 					xyz="0 0 0"
 					rpy="0 0 0" />
-				<geometry>
-					<mesh filename="package://mushr_description/meshes/base/tx2/mushr_base_tx2_collision.dae" />
-				</geometry>
-			</collision>
+				<mass
+					value="1.0" />
+				<inertia
+					ixx="1"
+					ixy="0"
+					ixz="0"
+					iyy="1"
+					iyz="0"
+					izz="1" />
+			</inertial>
+			<xacro:unless value="${platform_color == 'none' and inset_color == 'none'}">
+				<visual>
+					<origin
+						xyz="0 0 0"
+						rpy="0 0 0" />
+					<geometry>
+						<mesh filename="package://mushr_description/meshes/base/tx2/mushr_base_tx2_insets.stl" />
+					</geometry>
+					<material name="${inset_color}"/>
+				</visual>
+				<collision>
+					<origin
+						xyz="0 0 0"
+						rpy="0 0 0" />
+					<geometry>
+						<mesh filename="package://mushr_description/meshes/base/tx2/mushr_base_tx2_insets_collision.dae" />
+					</geometry>
+				</collision>
+			</xacro:unless>
 		</link>
 		<joint
@@ -60,4 +151,26 @@
 				link="base_link" />
 		</joint>
+		<joint
+			name="base_link_to_platform_link"
+			type="fixed">
+			<origin
+				xyz="0 0 0.0"
+				rpy="0 0 0" />
+			<parent
+				link="base_link" />
+			<child
+				link="platform_link" />
+		</joint>
+		<joint
+			name="base_link_to_insets_link"
+			type="fixed">
+			<origin
+				xyz="0 0 0.0"
+				rpy="0 0 0" />
+			<parent
+				link="base_link" />
+			<child
+				link="insets_link" />
+		</joint>
 	</xacro:macro>
 </robot>

File: mushr_description/robots/mushr_nano.urdf.xacro (robot description, xacro)
@@ -4,5 +4,7 @@
 	<xacro:include filename="mushr_ydlidar.urdf.xacro" />
 	<xacro:include filename="$(find realsense2_description)/urdf/_d435.urdf.xacro" />
-	<xacro:mushr_base_nano />
+	<xacro:arg name="platform_color" default="none"/>
+	<xacro:arg name="inset_color" default="none" />
+	<xacro:mushr_base_nano platform_color="$(arg platform_color)" inset_color="$(arg inset_color)"/>
 	<xacro:mushr_wheel prefix="front_left"  left="true" />
 	<xacro:mushr_wheel prefix="front_right" left="false"/>
@@ -15,7 +17,7 @@
 	<link name="front_left/wheel_steer_link"/>
 	<link name="front_right/wheel_steer_link" />
-        <joint
-	        name="front_left_wheel_steer"
-                type="revolute">
+  <joint
+    name="front_left_wheel_steer"
+    type="revolute">
 		<axis
 			xyz="0 0 1"/>
@@ -25,15 +27,15 @@
 			upper="1.57"
 			velocity="10.0"/>
-                <origin
-        	        xyz="0.1385 0.115 -0.045855"
-                        rpy="0 0 0" />
-                <parent
-                        link="base_link" />
-                <child
-                        link="front_left/wheel_steer_link" />
+    <origin
+      xyz="0.1385 0.115 -0.045855"
+      rpy="0 0 0" />
+    <parent
+    	link="base_link" />
+    <child
+      link="front_left/wheel_steer_link" />
 	</joint>
-        <joint
-	        name="front_right_wheel_steer"
-                type="revolute">
+	<joint
+		name="front_right_wheel_steer"
+    type="revolute">
 		<axis
 			xyz="0 0 1"/>
@@ -43,63 +45,63 @@
 			upper="1.57"
 			velocity="10.0"/>
-                <origin
-        	        xyz="0.1385 -0.115 -0.045855"
-                        rpy="0 0 0" />
-                <parent
-                        link="base_link" />
-                <child
-                        link="front_right/wheel_steer_link" />
+    <origin
+      xyz="0.1385 -0.115 -0.045855"
+      rpy="0 0 0" />
+    <parent
+      link="base_link" />
+    <child
+    	link="front_right/wheel_steer_link" />
 	</joint>
-        <joint
-	        name="front_left_wheel_throttle"
-                type="continuous">
+  <joint
+  	name="front_left_wheel_throttle"
+    type="continuous">
 		<axis
 			xyz="0 1 0"/>
-                <origin
-        	        xyz="0 0 0"
-                        rpy="0 0 0" />
-                <parent
-                        link="front_left/wheel_steer_link" />
-                <child
-                        link="front_left/wheel_link" />
+    <origin
+      xyz="0 0 0"
+      rpy="0 0 0" />
+    <parent
+    	link="front_left/wheel_steer_link" />
+    <child
+      link="front_left/wheel_link" />
 	</joint>
-        <joint
-	        name="front_right_wheel_throttle"
-                type="continuous">
+  <joint
+  	name="front_right_wheel_throttle"
+    type="continuous">
 		<axis
 			xyz="0 1 0"/>
-                <origin
-        	        xyz="0 0 0"
-                        rpy="0 0 0" />
-                <parent
-                        link="front_right/wheel_steer_link" />
-                <child
-                        link="front_right/wheel_link" />
+    <origin
+      xyz="0 0 0"
+      rpy="0 0 0" />
+    <parent
+    	link="front_right/wheel_steer_link" />
+    <child
+      link="front_right/wheel_link" />
 	</joint>
-        <joint
-	        name="back_left_wheel_throttle"
-                type="continuous">
+  <joint
+    name="back_left_wheel_throttle"
+    type="continuous">
 		<axis
 			xyz="0 1 0"/>
-                <origin
-        	        xyz="-0.158 0.115 -0.045855"
-                        rpy="0 0 0" />
-                <parent
-                        link="base_link" />
-                <child
-                        link="back_left/wheel_link" />
+    <origin
+      xyz="-0.158 0.115 -0.045855"
+      rpy="0 0 0" />
+    <parent
+      link="base_link" />
+    <child
+      link="back_left/wheel_link" />
 	</joint>
-        <joint
-	        name="back_right_wheel_throttle"
-                type="continuous">
+  <joint
+  	name="back_right_wheel_throttle"
+  	type="continuous">
 		<axis
 			xyz="0 1 0"/>
-                <origin
-        	        xyz="-0.158 -0.115 -0.045855"
-                        rpy="0 0 0" />
-                <parent
-                        link="base_link" />
-                <child
-                        link="back_right/wheel_link" />
+    <origin
+      xyz="-0.158 -0.115 -0.045855"
+      rpy="0 0 0" />
+    <parent
+      link="base_link" />
+    <child
+      link="back_right/wheel_link" />
 	</joint>
 	<joint

File: mushr_description/robots/mushr_tx2.urdf.xacro (robot description, xacro)
@@ -4,5 +4,7 @@
 	<xacro:include filename="mushr_ydlidar.urdf.xacro" />
 	<xacro:include filename="$(find realsense2_description)/urdf/_d435.urdf.xacro" />
-	<xacro:mushr_base_tx2 />
+	<xacro:arg name="platform_color" default="none"/>
+	<xacro:arg name="inset_color" default="none" />
+	<xacro:mushr_base_tx2 platform_color="$(arg platform_color)" inset_color="$(arg inset_color)"/>
 	<xacro:mushr_wheel prefix="front_left"  left="true" />
 	<xacro:mushr_wheel prefix="front_right" left="false"/>
@@ -15,7 +17,7 @@
 	<link name="front_left/wheel_steer_link"/>
 	<link name="front_right/wheel_steer_link" />
-        <joint
-	        name="front_left_wheel_steer"
-                type="revolute">
+  <joint
+  	name="front_left_wheel_steer"
+    type="revolute">
 		<axis
 			xyz="0 0 1"/>
@@ -25,15 +27,15 @@
 			upper="1.57"
 			velocity="10.0"/>
-                <origin
-        	        xyz="0.1385 0.115 -0.045855"
-                        rpy="0 0 0" />
-                <parent
-                        link="base_link" />
-                <child
-                        link="front_left/wheel_steer_link" />
+    <origin
+      xyz="0.1385 0.115 -0.045855"
+      rpy="0 0 0" />
+    <parent
+      link="base_link" />
+    <child
+      link="front_left/wheel_steer_link" />
 	</joint>
-        <joint
-	        name="front_right_wheel_steer"
-                type="revolute">
+  <joint
+  	name="front_right_wheel_steer"
+    type="revolute">
 		<axis
 			xyz="0 0 1"/>
@@ -43,63 +45,63 @@
 			upper="1.57"
 			velocity="10.0"/>
-                <origin
-        	        xyz="0.1385 -0.115 -0.045855"
-                        rpy="0 0 0" />
-                <parent
-                        link="base_link" />
-                <child
-                        link="front_right/wheel_steer_link" />
+		<origin
+		  xyz="0.1385 -0.115 -0.045855"
+		  rpy="0 0 0" />
+		<parent
+		  link="base_link" />
+		<child
+			link="front_right/wheel_steer_link" />
 	</joint>
-        <joint
-	        name="front_left_wheel_throttle"
-                type="continuous">
+  <joint
+    name="front_left_wheel_throttle"
+    type="continuous">
 		<axis
 			xyz="0 1 0"/>
-                <origin
-        	        xyz="0 0 0"
-                        rpy="0 0 0" />
-                <parent
-                        link="front_left/wheel_steer_link" />
-                <child
-                        link="front_left/wheel_link" />
+		<origin
+		  xyz="0 0 0"
+		  rpy="0 0 0" />
+		<parent
+		  link="front_left/wheel_steer_link" />
+		<child
+		  link="front_left/wheel_link" />
 	</joint>
-        <joint
-	        name="front_right_wheel_throttle"
-                type="continuous">
+  <joint
+    name="front_right_wheel_throttle"
+    type="continuous">
 		<axis
 			xyz="0 1 0"/>
-                <origin
-        	        xyz="0 0 0"
-                        rpy="0 0 0" />
-                <parent
-                        link="front_right/wheel_steer_link" />
-                <child
-                        link="front_right/wheel_link" />
+    <origin
+      xyz="0 0 0"
+      rpy="0 0 0" />
+    <parent
+      link="front_right/wheel_steer_link" />
+    <child
+      link="front_right/wheel_link" />
 	</joint>
-        <joint
-	        name="back_left_wheel_throttle"
-                type="continuous">
+  <joint
+    name="back_left_wheel_throttle"
+    type="continuous">
 		<axis
 			xyz="0 1 0"/>
-                <origin
-        	        xyz="-0.158 0.115 -0.045855"
-                        rpy="0 0 0" />
-                <parent
-                        link="base_link" />
-                <child
-                        link="back_left/wheel_link" />
+    <origin
+      xyz="-0.158 0.115 -0.045855"
+      rpy="0 0 0" />
+    <parent
+      link="base_link" />
+    <child
+      link="back_left/wheel_link" />
 	</joint>
-        <joint
-	        name="back_right_wheel_throttle"
-                type="continuous">
+  <joint
+	  name="back_right_wheel_throttle"
+	  type="continuous">
 		<axis
 			xyz="0 1 0"/>
-                <origin
-        	        xyz="-0.158 -0.115 -0.045855"
-                        rpy="0 0 0" />
-                <parent
-                        link="base_link" />
-                <child
-                        link="back_right/wheel_link" />
+    <origin
+      xyz="-0.158 -0.115 -0.045855"
+      rpy="0 0 0" />
+    <parent
+      link="base_link" />
+    <child
+      link="back_right/wheel_link" />
 	</joint>
 	<joint
