Commit message: testing swapping urdf files to fix localization issue

File: mushr_description/robots/mushr_base_nano.urdf.xacro (robot description, xacro)
@@ -33,40 +33,40 @@
 					izz="1" />
 			</inertial>
-			<xacro:if value="${platform_color == 'none' and inset_color == 'none'}">
-			<visual>
-					<origin
-						xyz="0 0 0"
-						rpy="0 0 0" />
-					<geometry>
-						<mesh filename="package://mushr_description/meshes/base/nano/mushr_base_nano.dae" />
-					</geometry>
-				</visual>
-				<collision>
-					<origin
-						xyz="0 0 0"
-						rpy="0 0 0" />
-					<geometry>
-						<mesh filename="package://mushr_description/meshes/base/nano/mushr_base_nano_collision.dae" />
-					</geometry>
-				</collision>
-			</xacro:if>
-			<xacro:unless value="${platform_color == 'none' and inset_color == 'none'}">
+				<xacro:if value="${platform_color == 'none' and inset_color == 'none'}">
 				<visual>
-					<origin
-						xyz="0 0 0"
-						rpy="0 0 0" />
-					<geometry>
-						<mesh filename="package://mushr_description/meshes/base/nano/mushr_base_nano_core.dae" />
-					</geometry>
-				</visual>
-				<collision>
-					<origin
-						xyz="0 0 0"
-						rpy="0 0 0" />
-					<geometry>
-						<mesh filename="package://mushr_description/meshes/base/nano/mushr_base_nano_core_collision.dae" />
-					</geometry>
-				</collision>
-			</xacro:unless>
+						<origin
+							xyz="0 0 0"
+							rpy="0 0 0" />
+						<geometry>
+							<mesh filename="package://mushr_description/meshes/base/nano/mushr_base_nano.dae" />
+						</geometry>
+					</visual>
+					<collision>
+						<origin
+							xyz="0 0 0"
+							rpy="0 0 0" />
+						<geometry>
+							<mesh filename="package://mushr_description/meshes/base/nano/mushr_base_nano_collision.dae" />
+						</geometry>
+					</collision>
+				</xacro:if>
+				<xacro:unless value="${platform_color == 'none' and inset_color == 'none'}">
+					<visual>
+						<origin
+							xyz="0 0 0"
+							rpy="0 0 0" />
+						<geometry>
+							<mesh filename="package://mushr_description/meshes/base/nano/mushr_base_nano_core.dae" />
+						</geometry>
+					</visual>
+					<collision>
+						<origin
+							xyz="0 0 0"
+							rpy="0 0 0" />
+						<geometry>
+							<mesh filename="package://mushr_description/meshes/base/nano/mushr_base_nano_core_collision.dae" />
+						</geometry>
+					</collision>
+				</xacro:unless>
 		</link>
 		<link name="platform_link">
@@ -85,23 +85,23 @@
 					izz="1" />
 			</inertial>
-			<xacro:unless value="${platform_color == 'none' and inset_color == 'none'}">
-				<visual>
-					<origin
-						xyz="0 0 0"
-						rpy="0 0 0" />
-					<geometry>
-						<mesh filename="package://mushr_description/meshes/base/nano/mushr_base_nano_platform.stl" />
-					</geometry>
-					<material name="${platform_color}"/>
-				</visual>
-				<collision>
-					<origin
-						xyz="0 0 0"
-						rpy="0 0 0" />
-					<geometry>
-						<mesh filename="package://mushr_description/meshes/base/nano/mushr_base_nano_platform_collision.dae" />
-					</geometry>
-				</collision>
-			</xacro:unless>
+				<xacro:unless value="${platform_color == 'none' and inset_color == 'none'}">
+					<visual>
+						<origin
+							xyz="0 0 0"
+							rpy="0 0 0" />
+						<geometry>
+							<mesh filename="package://mushr_description/meshes/base/nano/mushr_base_nano_platform.stl" />
+						</geometry>
+						<material name="${platform_color}"/>
+					</visual>
+					<collision>
+						<origin
+							xyz="0 0 0"
+							rpy="0 0 0" />
+						<geometry>
+							<mesh filename="package://mushr_description/meshes/base/nano/mushr_base_nano_platform_collision.dae" />
+						</geometry>
+					</collision>
+				</xacro:unless>
 		</link>
 		<link name="insets_link">
@@ -120,23 +120,23 @@
 					izz="1" />
 			</inertial>
-			<xacro:unless value="${platform_color == 'none' and inset_color == 'none'}">
-				<visual>
-					<origin
-						xyz="0 0 0"
-						rpy="0 0 0" />
-					<geometry>
-						<mesh filename="package://mushr_description/meshes/base/nano/mushr_base_nano_insets.stl" />
-					</geometry>
-					<material name="${inset_color}"/>
-				</visual>
-				<collision>
-					<origin
-						xyz="0 0 0"
-						rpy="0 0 0" />
-					<geometry>
-						<mesh filename="package://mushr_description/meshes/base/nano/mushr_base_nano_insets_collision.dae" />
-					</geometry>
-				</collision>
-			</xacro:unless>
+				<xacro:unless value="${platform_color == 'none' and inset_color == 'none'}">
+					<visual>
+						<origin
+							xyz="0 0 0"
+							rpy="0 0 0" />
+						<geometry>
+							<mesh filename="package://mushr_description/meshes/base/nano/mushr_base_nano_insets.stl" />
+						</geometry>
+						<material name="${inset_color}"/>
+					</visual>
+					<collision>
+						<origin
+							xyz="0 0 0"
+							rpy="0 0 0" />
+						<geometry>
+							<mesh filename="package://mushr_description/meshes/base/nano/mushr_base_nano_insets_collision.dae" />
+						</geometry>
+					</collision>
+				</xacro:unless>
 		</link>
 		<joint

File: mushr_description/robots/mushr_urdf_files/oldmushr_nano.urdf.xacro (robot description, xacro)
@@ -107,5 +107,5 @@
 	<joint
 		name="base_link_to_laser_link"
-		type="fixed">
+		type="fixed" >
 		<origin
 			xyz="-0.035325 0 0.10775"
